Commit message: Aruco Markers

File: robotino3_description/robotino/RobotinoModel/urdf/robotino.urdf (robot description, URDF)
Before this commit: robot robotino, 9 links, 8 joints
Links:
- added link camera_link_optical
Joints:
- added joint camera_optical_joint: type fixed, parent camera_link, child camera_link_optical, origin xyz=0 0 0 rpy=-1.570795 0 -1.570795
- joint camera_joint: origin xyz=0.044 0 0.07 rpy=0 0 1.570795 -> xyz=0.044 0 0.2 rpy=0 0 0

Commit message: ajusted parameters to be more in line with reality

File: robotino3_description/robotino/RobotinoModel/urdf/robotino.urdf (robot description, URDF)
Before this commit: robot robotino, 10 links, 9 joints
Joints:
- joint camera_joint: origin xyz=0.044 0 0.2 rpy=0 0 0 -> xyz=0.044 0 0.475 rpy=0 0 0
